Commit message: Adjust pitch

File: catkin_ws/src/mapping/urdf/goliath.urdf (robot description, URDF)
Before this commit: robot test_map, 4 links, 3 joints
Joints:
- joint t265_link_to_d455_link_joint: origin xyz=0.045 0 0.09 rpy=0 0.3 0 -> xyz=0.045 0 0.09 rpy=0 0.175 0

Commit message: Hmm let's increase pitch

File: catkin_ws/src/mapping/urdf/goliath.urdf (robot description, URDF)
Before this commit: robot test_map, 4 links, 3 joints
Joints:
- joint t265_link_to_d455_link_joint: origin xyz=0.045 0 0.09 rpy=0 0.175 0 -> xyz=0.045 0 0.09 rpy=0 0.218 0
